File: ac_current_sense.kicad_sch (KiCad schematic)
At the start: 23 parts, among them J5 IA+, J6 IA-, J7 IC+, J8 IB+, J9 IB-

Commit message: PCB V1
Parts:
- removed J5: IA+, symbol Connector_Generic:Conn_01x01
- removed J6: IA-, symbol Connector_Generic:Conn_01x01
- removed J7: IC+, symbol Connector_Generic:Conn_01x01
- removed J8: IB+, symbol Connector_Generic:Conn_01x01
- removed J9: IB-, symbol Connector_Generic:Conn_01x01
- added J20: AC Current Header, Connector_PinHeader_2.54mm:PinHeader_1x06_P2.54mm_Vertical, symbol Connector_Generic:Conn_01x06
- C10, C11, C12, C13, C14, C15: footprint CAPC220145_100N_KEM -> Capacitor_SMD:C_0805_2012Metric_Pad1.18x1.45mm_HandSolder
- R10, R11, R12, R13, R17, R18: value 2.4ohm RC0805FR-072R4L -> 2.4ohm; footprint RC0805FR-072R4L:RESC2012X60N -> Resistor_SMD:R_0805_2012Metric_Pad1.20x1.40mm_HandSolder
- R14, R15, R16, R19, R22: footprint RC0805N_YAG -> Resistor_SMD:R_0805_2012Metric_Pad1.20x1.40mm_HandSolder
- R20: value 1kohm RC0805FR-071KL -> 1kohm; footprint RC0805N_YAG -> Resistor_SMD:R_0805_2012Metric_Pad1.20x1.40mm_HandSolder
Connections:
- net IC+: now reaches R12.2, R16.2
- net IC+: now also J20.2 (Pin_2)
- net IA-: now reaches R11.1, R15.2
- net IA-: now also J20.5 (Pin_5)
- net IC-: now reaches R13.1, R22.2
- net IC-: now also J20.1 (Pin_1)
- net IA+: now reaches R10.2, R14.2
- net IA+: now also J20.6 (Pin_6)
- net IB+: now reaches R17.2, R19.2
- net IB+: now also J20.4 (Pin_4)
- net IB-: now reaches R18.1, R20.2
- net IB-: now also J20.3 (Pin_3)
