File: ac_voltage_sense.kicad_sch (KiCad schematic)
At the start: 13 parts, among them J11 UN, J2 UA, J3 UB, J4 UC

Commit message: PCB V1
Parts:
- C4, C5, C6: value 1800pF C0805C182G1HACTU -> 1800pF; footprint CAPC220145_100N_KEM -> Capacitor_SMD:C_0805_2012Metric_Pad1.18x1.45mm_HandSolder
- J11, J2, J3, J4: footprint (none) -> Connector:Banana_Jack_1Pin
- R1, R2, R3: value 4Mohm RMCF0805FT4M02 -> 4Mohm; footprint RES_RMCF0805_STP -> Resistor_SMD:R_0805_2012Metric_Pad1.20x1.40mm_HandSolder
- R4, R5, R6: value 16.9kohm RC0805FR-0716K9L -> 16.9kohm; footprint RC0805N_YAG -> Resistor_SMD:R_0805_2012Metric_Pad1.20x1.40mm_HandSolder
Connections:
- net GND: now also R6.2
Changed lines of the file:
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@@
+	)
+	(junction
+		(at 118.11 123.19)
+		(diameter 0)
+		(color 0 0 0 0)
 	)
 	(junction
@@
 	(wire
 		(pts
-			(xy 128.27 118.11) (xy 128.27 121.92)
+			(xy 128.27 118.11) (xy 128.27 123.19)
 		)
 		(stroke
@@
 	(wire
 		(pts
-			(xy 128.27 121.92) (xy 118.11 121.92)
+			(xy 128.27 123.19) (xy 118.11 123.19)
 		)
 		(stroke
@@
 		)
 	)
-	(hierarchical_label "V2P"
+	(global_label "V2P"
 		(shape output)
 		(at 133.35 73.66 0)
@@
 			(justify left)
 		)
-	)
-	(hierarchical_label "V3P"
+		(property "Intersheetrefs" "${INTERSHEET_REFS}"
+			(at 139.9033 73.66 0)
+			(effects
+				(font
+					(size 1.27 1.27)
+				)
+				(justify left)
+				(hide yes)
+			)
+		)
+	)
+	(global_label "V3P"
 		(shape output)
 		(at 134.62 105.41 0)
@@
 			(justify left)
 		)
-	)
-	(hierarchical_label "V1P"
+		(property "Intersheetrefs" "${INTERSHEET_REFS}"
+			(at 141.1733 105.41 0)
+			(effects
+				(font
+					(size 1.27 1.27)
+				)
+				(justify left)
+				(hide yes)
+			)
+		)
+	)
+	(global_label "V1P"
 		(shape output)
 		(at 132.08 41.91 0)
@@
 			(justify left)
 		)
+		(property "Intersheetrefs" "${INTERSHEET_REFS}"
+			(at 138.6333 41.91 0)
+			(effects
+				(font
+					(size 1.27 1.27)
+				)
+				(justify left)
+				(hide yes)
+			)
+		)
 	)
 	(symbol
@@
 			)
 		)
-		(property "Value" "4Mohm RMCF0805FT4M02"
+		(property "Value" "4Mohm"
 			(at 106.68 69.85 0)
 			(effects
@@
 			)
 		)
-		(property "Footprint" "RES_RMCF0805_STP"
+		(property "Footprint" "Resistor_SMD:R_0805_2012Metric_Pad1.20x1.40mm_HandSolder"
 			(at 100.33 73.66 0)
 			(effects
@@
 			)
 		)
-		(property "Value" "1800pF C0805C182G1HACTU"
+		(property "Value" "1800pF"
 			(at 130.81 83.8199 90)
 			(effects
@@
 			)
 		)
-		(property "Footprint" "CAPC220145_100N_KEM"
+		(property "Footprint" "Capacitor_SMD:C_0805_2012Metric_Pad1.18x1.45mm_HandSolder"
 			(at 127 86.36 0)
 			(effects
@@
 			)
 		)
-		(property "Value" "1800pF C0805C182G1HACTU"
+		(property "Value" "1800pF"
 			(at 132.08 115.5699 90)
 			(effects
@@
 			)
 		)
-		(property "Footprint" "CAPC220145_100N_KEM"
+		(property "Footprint" "Capacitor_SMD:C_0805_2012Metric_Pad1.18x1.45mm_HandSolder"
 			(at 128.27 118.11 0)
 			(effects
@@
 			)
 		)
-		(property "Footprint" ""
+		(property "Footprint" "Connector:Banana_Jack_1Pin"
 			(at 81.28 105.41 0)
 			(effects
@@
 			)
 		)
-		(property "Footprint" ""
+		(property "Footprint" "Connector:Banana_Jack_1Pin"
 			(at 82.55 130.81 0)
 			(effects
@@
 			)
 		)
-		(property "Value" "4Mohm RMCF0805FT4M02"
+		(property "Value" "4Mohm"
 			(at 109.22 101.6 0)
 			(effects
@@
 			)
 		)
-		(property "Footprint" "RES_RMCF0805_STP"
+		(property "Footprint" "Resistor_SMD:R_0805_2012Metric_Pad1.20x1.40mm_HandSolder"
 			(at 102.87 105.41 0)
 			(effects
@@
 		(on_board yes)
 		(dnp no)
-		(fields_autoplaced yes)
 		(property "Reference" "R4"
-			(at 118.11 50.7999 90)
+			(at 103.378 51.054 90)
 			(effects
 				(font
@@
 			)
 		)
-		(property "Value" "16.9kohm RC0805FR-0716K9L"
-			(at 118.11 53.3399 90)
+		(property "Value" "16.9kohm"
+			(at 103.378 53.594 90)
 			(effects
 				(font
@@
 			)
 		)
-		(property "Footprint" "RC0805N_YAG"
+		(property "Footprint" "Resistor_SMD:R_0805_2012Metric_Pad1.20x1.40mm_HandSolder"
 			(at 115.57 58.42 0)
 			(effects
@@
 			)
 		)
-		(property "Footprint" ""
+		(property "Footprint" "Connector:Banana_Jack_1Pin"
 			(at 78.74 41.91 0)
 			(effects
@@
 			)
 		)
-		(property "Footprint" ""
+		(property "Footprint" "Connector:Banana_Jack_1Pin"
 			(at 80.01 73.66 0)
 			(effects
@@
 	(symbol
 		(lib_id "power:GND")
-		(at 118.11 121.92 0)
+		(at 118.11 123.19 0)
 		(unit 1)
 		(exclude_from_sim no)
@@
 		(fields_autoplaced yes)
 		(property "Reference" "#PWR018"
+			(at 118.11 129.54 0)
+			(effects
+				(font
+					(size 1.27 1.27)
+				)
+				(hide yes)
+			)
+		)
+		(property "Value" "GND"
 			(at 118.11 128.27 0)
 			(effects
@@
 					(size 1.27 1.27)
 				)
-				(hide yes)
-			)
-		)
-		(property "Value" "GND"
-			(at 118.11 127 0)
-			(effects
-				(font
-					(size 1.27 1.27)
-				)
 			)
 		)
 		(property "Footprint" ""
-			(at 118.11 121.92 0)
+			(at 118.11 123.19 0)
 			(effects
 				(font
@@
 		)
 		(property "Datasheet" ""
-			(at 118.11 121.92 0)
+			(at 118.11 123.19 0)
 			(effects
 				(font
@@
 		)
 		(property "Description" "Power symbol creates a global label with name \"GND\" , ground"
-			(at 118.11 121.92 0)
+			(at 118.11 123.19 0)
 			(effects
 				(font
@@
 		(on_board yes)
 		(dnp no)
-		(fields_autoplaced yes)
 		(property "Reference" "R5"
-			(at 119.38 82.5499 90)
+			(at 104.394 81.534 90)
 			(effects
 				(font
@@
 			)
 		)
-		(property "Value" "16.9kohm RC0805FR-0716K9L"
-			(at 119.38 85.0899 90)
+		(property "Value" "16.9kohm"
+			(at 104.394 84.074 90)
 			(effects
 				(font
@@
 			)
 		)
-		(property "Footprint" "RC0805N_YAG"
+		(property "Footprint" "Resistor_SMD:R_0805_2012Metric_Pad1.20x1.40mm_HandSolder"
 			(at 116.84 90.17 0)
 			(effects
@@
 		(on_board yes)
 		(dnp no)
-		(fields_autoplaced yes)
 		(property "Reference" "R6"
-			(at 120.65 115.5699 90)
+			(at 105.664 114.3 90)
 			(effects
 				(font
@@
 			)
 		)
-		(property "Value" "16.9kohm RC0805FR-0716K9L"
-			(at 120.65 118.1099 90)
+		(property "Value" "16.9kohm"
+			(at 105.664 116.84 90)
 			(effects
 				(font
@@
 			)
 		)
-		(property "Footprint" "RC0805N_YAG"
+		(property "Footprint" "Resistor_SMD:R_0805_2012Metric_Pad1.20x1.40mm_HandSolder"
 			(at 118.11 123.19 0)
 			(effects
@@
 		(on_board yes)
 		(dnp no)
-		(fields_autoplaced yes)
 		(property "Reference" "R1"
 			(at 105.41 35.56 0)
@@
 			)
 		)
-		(property "Value" "4Mohm RMCF0805FT4M02"
+		(property "Value" "4Mohm"
 			(at 105.41 38.1 0)
 			(effects
@@
 			)
 		)
-		(property "Footprint" "RES_RMCF0805_STP"
+		(property "Footprint" "Resistor_SMD:R_0805_2012Metric_Pad1.20x1.40mm_HandSolder"
 			(at 99.06 41.91 0)
 			(effects
@@
 			)
 		)
-		(property "Value" "1800pF C0805C182G1HACTU"
+		(property "Value" "1800pF"
 			(at 129.54 52.0699 90)
 			(effects
@@
 			)
 		)
-		(property "Footprint" "CAPC220145_100N_KEM"
+		(property "Footprint" "Capacitor_SMD:C_0805_2012Metric_Pad1.18x1.45mm_HandSolder"
 			(at 125.73 54.61 0)
 			(effects
