File: dc_sense.kicad_sch (KiCad schematic)
At the start: 3 parts, among them U2 TMCS1108A3UQDR

Commit message: PCB V1
Parts:
- added J12: DC_I_P, Connector:Banana_Jack_1Pin, symbol Connector_Generic:Conn_01x01
- added J13: DC_I_N, Connector:Banana_Jack_1Pin, symbol Connector_Generic:Conn_01x01
- added J15: DC Current and Voltage Sensors, Connector_PinHeader_2.54mm:PinHeader_1x02_P2.54mm_Vertical, symbol Connector:Conn_01x02_Socket
- R23, R24: footprint (none) -> Resistor_SMD:R_0805_2012Metric_Pad1.20x1.40mm_HandSolder
- U2: footprint D0008A-IPC_A -> TMCS1108A3U:D0008A-IPC_A
Connections:
- net VDC is gone; now on net DC_I_P: R23.1
- net DC_I_N: now also J13.1 (Pin_1)
- net DC_I_P: now also J12.1 (Pin_1)
- net DC_I_SENSE_V: now also J15.1 (Pin_1)
- net DC_V_SENSE: now also J15.2 (Pin_2)
- net +3.3VA renamed +3.3V
Changed lines of the file:
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@@
 	(wire
 		(pts
-			(xy 82.55 57.15) (xy 90.17 57.15)
+			(xy 74.93 57.15) (xy 90.17 57.15)
 		)
 		(stroke
@@
 	(wire
 		(pts
-			(xy 82.55 69.85) (xy 90.17 69.85)
+			(xy 74.93 69.85) (xy 90.17 69.85)
 		)
 		(stroke
@@
 	(wire
 		(pts
-			(xy 176.53 52.07) (xy 176.53 50.8)
+			(xy 176.53 45.72) (xy 176.53 52.07)
 		)
 		(stroke
@@
 	(text "60V DC Voltage Sense"
 		(exclude_from_sim no)
-		(at 175.006 42.418 0)
+		(at 176.53 35.306 0)
 		(effects
 			(font
@@
 				(size 1.27 1.27)
 			)
+		)
+	)
+	(label "DC_V_SENSE"
+		(at 146.05 82.55 180)
+		(fields_autoplaced yes)
+		(effects
+			(font
+				(size 1.27 1.27)
+			)
+			(justify right bottom)
+		)
+	)
+	(label "DC_I_SENSE_V"
+		(at 129.54 60.96 0)
+		(fields_autoplaced yes)
+		(effects
+			(font
+				(size 1.27 1.27)
+			)
+			(justify left bottom)
 		)
 	)
@@
 		)
 	)
-	(hierarchical_label "DC_I_SENSE_V"
-		(shape output)
-		(at 129.54 60.96 0)
-		(fields_autoplaced yes)
-		(effects
-			(font
-				(size 1.27 1.27)
-			)
-			(justify left)
-		)
-	)
-	(hierarchical_label "DC_V_SENSE"
-		(shape output)
+	(label "DC_I_SENSE_V"
+		(at 146.05 80.01 180)
+		(fields_autoplaced yes)
+		(effects
+			(font
+				(size 1.27 1.27)
+			)
+			(justify right bottom)
+		)
+	)
+	(label "VDC+"
+		(at 74.93 57.15 0)
+		(fields_autoplaced yes)
+		(effects
+			(font
+				(size 1.27 1.27)
+			)
+			(justify left bottom)
+		)
+	)
+	(label "DC_V_SENSE"
 		(at 180.34 60.96 0)
 		(fields_autoplaced yes)
@@
 				(size 1.27 1.27)
 			)
-			(justify left)
-		)
-	)
-	(symbol
-		(lib_id "power:VDC")
-		(at 176.53 50.8 0)
-		(unit 1)
-		(exclude_from_sim no)
-		(in_bom yes)
-		(on_board yes)
-		(dnp no)
-		(fields_autoplaced yes)
-		(property "Reference" "#PWR021"
-			(at 176.53 54.61 0)
-			(effects
-				(font
-					(size 1.27 1.27)
-				)
-				(hide yes)
-			)
-		)
-		(property "Value" "VDC"
-			(at 176.53 45.72 0)
-			(effects
-				(font
-					(size 1.27 1.27)
-				)
-			)
-		)
-		(property "Footprint" ""
-			(at 176.53 50.8 0)
-			(effects
-				(font
-					(size 1.27 1.27)
-				)
-				(hide yes)
-			)
-		)
-		(property "Datasheet" ""
-			(at 176.53 50.8 0)
-			(effects
-				(font
-					(size 1.27 1.27)
-				)
-				(hide yes)
-			)
-		)
-		(property "Description" "Power symbol creates a global label with name \"VDC\""
-			(at 176.53 50.8 0)
-			(effects
-				(font
-					(size 1.27 1.27)
-				)
-				(hide yes)
-			)
-		)
-		(pin "1"
-		)
-		(instances
-			(project "SeniorProjectVSC-3phSensor"
-				(path "/92b98703-669a-49fb-bccd-3cc8cbdd124b/ef3b8b51-e9e1-444c-9195-06111c21df75"
-					(reference "#PWR021")
-					(unit 1)
-				)
-			)
+			(justify left bottom)
+		)
+	)
+	(label "VDC+"
+		(at 176.53 45.72 0)
+		(fields_autoplaced yes)
+		(effects
+			(font
+				(size 1.27 1.27)
+			)
+			(justify left bottom)
 		)
 	)
@@
 			)
 		)
-		(property "Footprint" ""
+		(property "Footprint" "Resistor_SMD:R_0805_2012Metric_Pad1.20x1.40mm_HandSolder"
 			(at 177.546 56.134 90)
 			(effects
@@
 			)
 		)
-		(property "Footprint" ""
+		(property "Footprint" "Resistor_SMD:R_0805_2012Metric_Pad1.20x1.40mm_HandSolder"
 			(at 177.546 66.294 90)
 			(effects
@@
 	)
 	(symbol
+		(lib_id "Connector:Conn_01x02_Socket")
+		(at 151.13 80.01 0)
+		(unit 1)
+		(exclude_from_sim no)
+		(in_bom yes)
+		(on_board yes)
+		(dnp no)
+		(fields_autoplaced yes)
+		(property "Reference" "J15"
+			(at 152.4 80.0099 0)
+			(effects
+				(font
+					(size 1.27 1.27)
+				)
+				(justify left)
+			)
+		)
+		(property "Value" "DC Current and Voltage Sensors"
+			(at 152.4 82.5499 0)
+			(effects
+				(font
+					(size 1.27 1.27)
+				)
+				(justify left)
+			)
+		)
+		(property "Footprint" "Connector_PinHeader_2.54mm:PinHeader_1x02_P2.54mm_Vertical"
+			(at 151.13 80.01 0)
+			(effects
+				(font
+					(size 1.27 1.27)
+				)
+				(hide yes)
+			)
+		)
+		(property "Datasheet" "~"
+			(at 151.13 80.01 0)
+			(effects
+				(font
+					(size 1.27 1.27)
+				)
+				(hide yes)
+			)
+		)
+		(property "Description" "Generic connector, single row, 01x02, script generated"
+			(at 151.13 80.01 0)
+			(effects
+				(font
+					(size 1.27 1.27)
+				)
+				(hide yes)
+			)
+		)
+		(pin "1"
+		)
+		(pin "2"
+		)
+		(instances
+			(project "SeniorProjectVSC-3phSensor"
+				(path "/92b98703-669a-49fb-bccd-3cc8cbdd124b/ef3b8b51-e9e1-444c-9195-06111c21df75"
+					(reference "J15")
+					(unit 1)
+				)
+			)
+		)
+	)
+	(symbol
 		(lib_id "TMCS1108A3UQDR:TMCS1108A3UQDR")
 		(at 90.17 55.88 0)
@@
 			)
 		)
-		(property "Footprint" "D0008A-IPC_A"
+		(property "Footprint" "TMCS1108A3U:D0008A-IPC_A"
 			(at 90.17 55.88 0)
 			(effects
@@
 	)
 	(symbol
+		(lib_id "Connector_Generic:Conn_01x01")
+		(at 69.85 57.15 180)
+		(unit 1)
+		(exclude_from_sim no)
+		(in_bom yes)
+		(on_board yes)
+		(dnp no)
+		(fields_autoplaced yes)
+		(property "Reference" "J12"
+			(at 69.85 50.8 0)
+			(effects
+				(font
+					(size 1.27 1.27)
+				)
+			)
+		)
+		(property "Value" "DC_I_P"
+			(at 69.85 53.34 0)
+			(effects
+				(font
+					(size 1.27 1.27)
+				)
+			)
+		)
+		(property "Footprint" "Connector:Banana_Jack_1Pin"
+			(at 69.85 57.15 0)
+			(effects
+				(font
+					(size 1.27 1.27)
+				)
+				(hide yes)
+			)
+		)
+		(property "Datasheet" "~"
+			(at 69.85 57.15 0)
+			(effects
+				(font
+					(size 1.27 1.27)
+				)
+				(hide yes)
+			)
+		)
+		(property "Description" "Generic connector, single row, 01x01, script generated (kicad-library-utils/schlib/autogen/connector/)"
+			(at 69.85 57.15 0)
+			(effects
+				(font
+					(size 1.27 1.27)
+				)
+				(hide yes)
+			)
+		)
+		(pin "1"
+		)
+		(instances
+			(project "SeniorProjectVSC-3phSensor"
+				(path "/92b98703-669a-49fb-bccd-3cc8cbdd124b/ef3b8b51-e9e1-444c-9195-06111c21df75"
+					(reference "J12")
+					(unit 1)
+				)
+			)
+		)
+	)
+	(symbol
 		(lib_id "power:GND")
 		(at 176.53 72.39 0)
@@
 	)
 	(symbol
+		(lib_id "Connector_Generic:Conn_01x01")
+		(at 69.85 69.85 180)
+		(unit 1)
+		(exclude_from_sim no)
+		(in_bom yes)
+		(on_board yes)
+		(dnp no)
+		(fields_autoplaced yes)
+		(property "Reference" "J13"
+			(at 69.85 63.5 0)
+			(effects
+				(font
+					(size 1.27 1.27)
+				)
+			)
+		)
+		(property "Value" "DC_I_N"
+			(at 69.85 66.04 0)
+			(effects
+				(font
+					(size 1.27 1.27)
+				)
+			)
+		)
+		(property "Footprint" "Connector:Banana_Jack_1Pin"
+			(at 69.85 69.85 0)
+			(effects
+				(font
+					(size 1.27 1.27)
+				)
+				(hide yes)
+			)
+		)
+		(property "Datasheet" "~"
+			(at 69.85 69.85 0)
+			(effects
+				(font
+					(size 1.27 1.27)
+				)
+				(hide yes)
+			)
+		)
+		(property "Description" "Generic connector, single row, 01x01, script generated (kicad-library-utils/schlib/autogen/connector/)"
+			(at 69.85 69.85 0)
+			(effects
+				(font
+					(size 1.27 1.27)
+				)
+				(hide yes)
+			)
+		)
+		(pin "1"
+		)
+		(instances
+			(project "SeniorProjectVSC-3phSensor"
+				(path "/92b98703-669a-49fb-bccd-3cc8cbdd124b/ef3b8b51-e9e1-444c-9195-06111c21df75"
+					(reference "J13")
+					(unit 1)
+				)
+			)
+		)
+	)
+	(symbol
 		(lib_id "power:GND")
 		(at 129.54 71.12 0)
@@
 			)
 		)
-		(property "Value" "+3.3VA"
+		(property "Value" "+3.3V"
 			(at 129.54 50.8 0)
 			(effects
